Commit message: Removed (practically) invisible geometry on the wheels and reduced the memory footprint of the rover by reusing meshes where possible. Also changed the motor effort and speed values to reflect the capabilities of the motors to be put on the actual rover.

File: models/rover/TARS_V2.urdf (robot description, URDF)
Before this commit: robot TARS_V2, 12 links, 11 joints
Links:
- link link_suspension_backleft: geometry collision box size=0.27135 0.0381 0.14844; visual mesh filename=..\meshes\stl\TARS.V2.Suspension.001.stl scale=-0.001 0.001 0.001
- link link_suspension_backright: geometry collision box size=0.27135 0.0381 0.14844; visual mesh filename=..\meshes\stl\TARS.V2.Suspension.001.stl scale=0.001 0.001 0.001
- link link_suspension_frontright: geometry collision box size=0.27134 0.0381 0.14845; visual mesh filename=..\meshes\stl\TARS.V2.Suspension.001.stl scale=0.001 -0.001 0.001
- link link_wheel_backleft: geometry collision sphere radius=0.15989; visual mesh filename=..\meshes\stl\TARS.V2.Wheel.001.stl scale=0.001 0.001 0.001
- link link_wheel_backright: geometry collision sphere radius=0.15989; visual mesh filename=..\meshes\stl\TARS.V2.Wheel.001.stl scale=0.001 0.001 0.001
- link link_wheel_frontright: geometry collision sphere radius=0.15989; visual mesh filename=..\meshes\stl\TARS.V2.Wheel.001.stl scale=0.001 0.001 0.001

Commit message: Fixed rover URDF

File: models/rover/TARS_V2.urdf (robot description, URDF)
Before this commit: robot TARS_V2, 12 links, 11 joints
Links:
- link link_chassis: geometry collision box size=0.63 0.48 0.29562; visual mesh filename=model://rover/meshes/stl/TARS.V2.Chassis.stl scale=0.001 0.001 0.001
- link link_suspension_backleft: geometry collision box size=0.27135 0.0381 0.14844; visual mesh filename=model://rover/meshes/stl/TARS.V2.Suspension.001.stl scale=-0.001 0.001 0.001
- link link_suspension_backright: geometry collision box size=0.27135 0.0381 0.14844; visual mesh filename=model://rover/meshes/stl/TARS.V2.Suspension.001.stl scale=0.001 0.001 0.001
- link link_suspension_frontleft: geometry collision box size=0.27135 0.0381 0.14844; visual mesh filename=model://rover/meshes/stl/TARS.V2.Suspension.001.stl scale=0.001 0.001 0.001
- link link_suspension_frontright: geometry collision box size=0.27134 0.0381 0.14845; visual mesh filename=model://rover/meshes/stl/TARS.V2.Suspension.001.stl scale=0.001 -0.001 0.001
- link link_wheel_backleft: geometry collision sphere radius=0.15989; visual mesh filename=model://rover/meshes/stl/TARS.V2.Wheel.001.stl scale=0.001 0.001 0.001
- link link_wheel_backright: geometry collision sphere radius=0.15989; visual mesh filename=model://rover/meshes/stl/TARS.V2.Wheel.001.stl scale=0.001 0.001 0.001
- link link_wheel_frontleft: geometry collision sphere radius=0.15989; visual mesh filename=model://rover/meshes/stl/TARS.V2.Wheel.001.stl scale=0.001 0.001 0.001
- link link_wheel_frontright: geometry collision sphere radius=0.15989; visual mesh filename=model://rover/meshes/stl/TARS.V2.Wheel.001.stl scale=0.001 0.001 0.001

File: models/rover_simple/TARS_V2_Simple.urdf (robot description, URDF)
Before this commit: robot TARS_V2, 12 links, 11 joints
Links:
- link link_wheel_frontleft: geometry collision sphere radius=0.15989; visual sphere radius=0.15989
