Commit message: Change link_chassis to base_link and wheel joints to type revolute in TARS_V2_Simple.urdf

File: models/rover_simple/TARS_V2_Simple.urdf (robot description, URDF)
Before this commit: robot TARS_V2, 12 links, 11 joints
Links:
- removed link link_chassis
- added link base_link, mass 30.0; collision box size=0.63 0.48 0.29562; visual box size=0.63 0.48 0.29563
Joints:
- joint link_camera_back: parent link_chassis -> base_link
- joint link_camera_depth: parent link_chassis -> base_link
- joint link_camera_front: parent link_chassis -> base_link
- joint link_suspension_backleft: parent link_chassis -> base_link
- joint link_suspension_backright: parent link_chassis -> base_link
- joint link_suspension_frontleft: parent link_chassis -> base_link
- joint link_suspension_frontright: parent link_chassis -> base_link
- joint link_wheel_backleft: limit (none) -> effort=100 velocity=100; type floating -> revolute
- joint link_wheel_backright: limit (none) -> effort=100 velocity=100; type floating -> revolute
- joint link_wheel_frontleft: limit (none) -> effort=100 velocity=100; type floating -> revolute
- joint link_wheel_frontright: limit (none) -> effort=100 velocity=100; type floating -> revolute
