Commit message: Move models and worlds into ros package

File: simulator/models/rover_simple/TARS_V2_Simple.urdf (robot description, URDF)
Before this commit: robot TARS_V2, 12 links, 11 joints
Joints:
- joint link_wheel_backleft: type revolute -> continuous
- joint link_wheel_backright: type revolute -> continuous
- joint link_wheel_frontleft: type revolute -> continuous
- joint link_wheel_frontright: type revolute -> continuous
