Commit message: Change model to unsimplified in gazebo.launch and set correct wheel rotation axis for unsimplified model

File: simulator/models/rover/TARS_V2.urdf (robot description, URDF)
Before this commit: robot TARS_V2, 12 links, 11 joints
Links:
- link link_chassis: geometry collision box size=0.63 0.48 0.29562; visual mesh filename=package://simulator/models/rover/meshes/stl/TARS.V2.Chassis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 scale=0.001 0.001 0.001
- link link_suspension_backleft: geometry collision box size=0.27135 0.0381 0.14844; visual mesh filename=package://simulator/models/rover/meshes/stl/TARS.V2.Suspens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 scale=0.001 0.001 0.001
- link link_suspension_backright: geometry collision box size=0.27135 0.0381 0.14844; visual mesh filename=package://simulator/models/rover/meshes/stl/TARS.V2.Suspens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 scale=0.001 0.001 0.001
- link link_suspension_frontleft: geometry collision box size=0.27135 0.0381 0.14844; visual mesh filename=package://simulator/models/rover/meshes/stl/TARS.V2.Suspens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 scale=0.001 0.001 0.001
- link link_suspension_frontright: geometry collision box size=0.27134 0.0381 0.14845; visual mesh filename=package://simulator/models/rover/meshes/stl/TARS.V2.Suspens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 scale=0.001 0.001 0.001
- link link_wheel_backleft: geometry collision sphere radius=0.15989; visual mesh filename=package://simulator/models/rover/meshes/stl/TARS.V2.Wheel.0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 scale=0.001 0.001 0.001
- link link_wheel_backright: geometry collision sphere radius=0.15989; visual mesh filename=package://simulator/models/rover/meshes/stl/TARS.V2.Wheel.0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 scale=0.001 0.001 0.001
- link link_wheel_frontleft: geometry collision sphere radius=0.15989; visual mesh filename=package://simulator/models/rover/meshes/stl/TARS.V2.Wheel.0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 scale=0.001 0.001 0.001
- link link_wheel_frontright: geometry collision sphere radius=0.15989; visual mesh filename=package://simulator/models/rover/meshes/stl/TARS.V2.Wheel.0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 scale=0.001 0.001 0.001
Joints:
- joint link_wheel_backleft: axis (none) -> 0 1 0; type floating -> continuous
- joint link_wheel_backright: axis (none) -> 0 1 0; type floating -> continuous
- joint link_wheel_frontleft: axis (none) -> 0 1 0; type floating -> continuous
- joint link_wheel_frontright: axis (none) -> 0 1 0; type floating -> continuous
