Commit message: limits set, but not accounting for physical collisions

File: spear_simulator/models/rover/arm.urdf (robot description, URDF)
Before this commit: robot arm, 7 links, 6 joints
Joints:
- joint shoulder: limit lower=-0.41 upper=2.15 effort=1 velocity=0.5 -> lower=0.78 upper=2.15 effort=1 velocity=0.5

Commit message: implement slim arm design with controller in rviz. mapper.py needs to be debugged.

File: spear_simulator/models/rover/arm.urdf (robot description, URDF)
Before this commit: robot arm, 7 links, 6 joints
Links:
- removed link hand
- removed link rotate
- added link palm
- added link wrist
Joints:
- removed joint elbow
- removed joint knuckle
- removed joint rotate
- removed joint shoulder
- removed joint shoulder_lift
- removed joint wrist
- added joint elbow_pitch: type revolute, parent bicep, child forearm, origin xyz=0 0 ${bicep_length} rpy=0 0 0, axis 0 1 0, limit lower=-2.7 upper=1.54 effort=1 velocity=0.5
- added joint grab: type revolute, parent palm, child finger, origin xyz=0 0 ${hand_length/3}, axis 1 0 0, limit lower=-1 upper=1 effort=1 velocity=0.5
- added joint shoulder_pitch: type revolute, parent shoulder, child bicep, origin xyz=0 0 ${shoulder_height} rpy=0 0 0, axis 0 1 0, limit lower=0.78 upper=2.15 effort=1 velocity=0.5
- added joint shoulder_yaw: type revolute, parent base_link, child shoulder, origin xyz=0 0 0 rpy=0 0 0, axis 0 0 1, limit lower=-1.58 upper=1.58 effort=1 velocity=0.5
- added joint wrist_pitch: type revolute, parent forearm, child wrist, origin xyz=0 0 ${forearm_length/5} rpy=0 0 0, axis 0 1 0, limit lower=-2.09 upper=2.09 effort=1 velocity=0.5
- added joint wrist_roll: type revolute, parent wrist, child palm, origin xyz=0 0 ${forearm_length/4} rpy=0 0 0, axis 0 0 1, limit lower=-3 upper=3 effort=1 velocity=0.5
