Commit message: Fix errors in simulator that were caused by the merge
Launch files and the model were still searching for a package called
"simulator". We named the package to "spear_simulator".

File: spear_simulator/models/rover/TARS_V2.urdf (robot description, URDF)
Before this commit: robot TARS_V2, 12 links, 11 joints
Links:
- link link_chassis: geometry collision box size=0.63 0.48 0.29562; visual mesh filename=package://spear_simulator/models/rover/meshes/stl/TARS.V2.C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 scale=0.001 0.001 0.001
- link link_suspension_backleft: geometry collision box size=0.27135 0.0381 0.14844; visual mesh filename=package://spear_simulator/models/rover/meshes/stl/TARS.V2.S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 scale=0.001 0.001 0.001
- link link_suspension_backright: geometry collision box size=0.27135 0.0381 0.14844; visual mesh filename=package://spear_simulator/models/rover/meshes/stl/TARS.V2.S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 scale=0.001 0.001 0.001
- link link_suspension_frontleft: geometry collision box size=0.27135 0.0381 0.14844; visual mesh filename=package://spear_simulator/models/rover/meshes/stl/TARS.V2.S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 scale=0.001 0.001 0.001
- link link_suspension_frontright: geometry collision box size=0.27134 0.0381 0.14845; visual mesh filename=package://spear_simulator/models/rover/meshes/stl/TARS.V2.S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 scale=0.001 0.001 0.001
- link link_wheel_backleft: geometry collision sphere radius=0.15989; visual mesh filename=package://spear_simulator/models/rover/meshes/stl/TARS.V2.W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 scale=0.001 0.001 0.001
- link link_wheel_backright: geometry collision sphere radius=0.15989; visual mesh filename=package://spear_simulator/models/rover/meshes/stl/TARS.V2.W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 scale=0.001 0.001 0.001
- link link_wheel_frontleft: geometry collision sphere radius=0.15989; visual mesh filename=package://spear_simulator/models/rover/meshes/stl/TARS.V2.W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 scale=0.001 0.001 0.001
- link link_wheel_frontright: geometry collision sphere radius=0.15989; visual mesh filename=package://spear_simulator/models/rover/meshes/stl/TARS.V2.W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 scale=0.001 0.001 0.001

Commit message: Rename link_chassis to base_link since tf expects the name 'base link'

File: spear_simulator/models/rover/TARS_V2.urdf (robot description, URDF)
Before this commit: robot TARS_V2, 12 links, 11 joints
Links:
- removed link link_chassis
- added link base_link, mass 30.0; collision box size=0.63 0.48 0.29562; visual mesh filename=package://spear_simulator/models/rover/meshes/stl/TARS.V2.C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 scale=0.001 0.001 0.001
Joints:
- joint link_camera_back: parent link_chassis -> base_link
- joint link_camera_depth: parent link_chassis -> base_link
- joint link_camera_front: parent link_chassis -> base_link
- joint link_suspension_backleft: parent link_chassis -> base_link
- joint link_suspension_backright: parent link_chassis -> base_link
- joint link_suspension_frontleft: parent link_chassis -> base_link
- joint link_suspension_frontright: parent link_chassis -> base_link

Commit message: Change roll of depth camera joint so that it is facing forwards

File: spear_simulator/models/rover/TARS_V2.urdf (robot description, URDF)
Before this commit: robot TARS_V2, 12 links, 11 joints
Joints:
- joint link_camera_depth: origin xyz=0.315 1e-05 0.3439 rpy=0 1.5708 0 -> xyz=0.315 1e-05 0.3439 rpy=0 0 0

Commit message: naming for links is consistent

File: spear_simulator/models/rover/TARS_V2.urdf (robot description, URDF)
Before this commit: robot TARS_V2, 12 links, 11 joints
Links:
- removed link link_wheel_backleft
- removed link link_wheel_backright
- removed link link_wheel_frontleft
- removed link link_wheel_frontright
- added link /CASE/controller/velocity/link_wheel_backleft, mass 1.5; collision sphere radius=0.15989; visual mesh filename=package://spear_simulator/models/rover/meshes/stl/TARS.V2.W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 scale=0.001 0.001 0.001
- added link /CASE/controller/velocity/link_wheel_backright, mass 1.5; collision sphere radius=0.15989; visual mesh filename=package://spear_simulator/models/rover/meshes/stl/TARS.V2.W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 scale=0.001 0.001 0.001
- added link /CASE/controller/velocity/link_wheel_frontleft, mass 1.5; collision sphere radius=0.15989; visual mesh filename=package://spear_simulator/models/rover/meshes/stl/TARS.V2.W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 scale=0.001 0.001 0.001
- added link /CASE/controller/velocity/link_wheel_frontright, mass 1.5; collision sphere radius=0.15989; visual mesh filename=package://spear_simulator/models/rover/meshes/stl/TARS.V2.W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 scale=0.001 0.001 0.001
Joints:
- removed joint link_wheel_backleft
- removed joint link_wheel_backright
- removed joint link_wheel_frontleft
- removed joint link_wheel_frontright
- added joint /CASE/controller/velocity/link_wheel_backleft: type continuous, parent link_suspension_backleft, child /CASE/controller/velocity/link_wheel_backleft, origin xyz=-0.21346 0.01924 -0.08012 rpy=0 0 0, axis 0 1 0
- added joint /CASE/controller/velocity/link_wheel_backright: type continuous, parent link_suspension_backright, child /CASE/controller/velocity/link_wheel_backright, origin xyz=-0.21346 -0.01886 -0.08012 rpy=0 0 0, axis 0 1 0
- added joint /CASE/controller/velocity/link_wheel_frontleft: type continuous, parent link_suspension_frontleft, child /CASE/controller/velocity/link_wheel_frontleft, origin xyz=0.21346 0.01886 -0.08012 rpy=0 0 0, axis 0 1 0
- added joint /CASE/controller/velocity/link_wheel_frontright: type continuous, parent link_suspension_frontright, child /CASE/controller/velocity/link_wheel_frontright, origin xyz=0.21345 -0.01924 -0.08014 rpy=0 0 0, axis 0 1 0

Commit message: Add imu_link to urdf

File: spear_simulator/models/rover/TARS_V2.urdf (robot description, URDF)
Before this commit: robot TARS_V2, 12 links, 11 joints
Links:
- added link imu_link
Joints:
- added joint imu_link: type fixed, parent base_link, child imu_link, origin xyz=0 0 0.2 rpy=0 0 0

Commit message: multiply the wheel-links in the urdf y-axis values  by -1 to correct opposite direction of odometry vector

File: spear_simulator/models/rover/TARS_V2.urdf (robot description, URDF)
Before this commit: robot TARS_V2, 13 links, 12 joints
Joints:
- joint link_wheel_backleft: axis 0 1 0 -> 0 -1 0
- joint link_wheel_backright: axis 0 1 0 -> 0 -1 0
- joint link_wheel_frontleft: axis 0 1 0 -> 0 -1 0
- joint link_wheel_frontright: axis 0 1 0 -> 0 -1 0

Commit message: Set ekf param two_d_mode to true and set wheel y axes back to +1

File: spear_simulator/models/rover/TARS_V2.urdf (robot description, URDF)
Before this commit: robot TARS_V2, 13 links, 12 joints
Joints:
- joint link_wheel_backleft: axis 0 -1 0 -> 0 1 0
- joint link_wheel_backright: axis 0 -1 0 -> 0 1 0
- joint link_wheel_frontleft: axis 0 -1 0 -> 0 1 0
- joint link_wheel_frontright: axis 0 -1 0 -> 0 1 0

Commit message: Restructure the launch files

File: spear_simulator/models/rover/TARS_V2.urdf (robot description, URDF)
Before this commit: robot TARS_V2, 13 links, 12 joints
Joints:
- joint link_camera_depth: origin xyz=0.315 1e-05 0.3439 rpy=0 0 0 -> xyz=0.3 0 0.2 rpy=0 0 0

Commit message: Define camera_depth_optical_frame within the robot model

File: spear_simulator/models/rover/TARS_V2.urdf (robot description, URDF)
Before this commit: robot TARS_V2, 13 links, 12 joints
Links:
- added link camera_depth_optical_frame
Joints:
- added joint camera_depth_optical_frame: type fixed, parent base_link, child camera_depth_optical_frame, origin xyz=0 0 0 rpy=${-M_PI/2} 0 ${-M_PI/2}

Commit message: Fix depth camera position

File: spear_simulator/models/rover/TARS_V2.urdf (robot description, URDF)
Before this commit: robot TARS_V2, 14 links, 13 joints
Joints:
- joint camera_depth_optical_frame: parent base_link -> link_camera_depth

Commit message: Commit changes and sort it out later

File: spear_simulator/models/rover/TARS_V2.urdf (robot description, URDF)
Before this commit: robot TARS_V2, 14 links, 13 joints
Links:
- link base_link: mass 30.0 -> None

Commit message: Changes

File: spear_simulator/models/rover/TARS_V2.urdf (robot description, URDF)
Before this commit: robot TARS_V2, 14 links, 13 joints
Links:
- added link zed_camera_center; visual mesh filename=package://zed_wrapper/urdf/models/ZED.stl
- added link zed_left_camera_frame
- added link zed_left_camera_optical_frame
- added link zed_right_camera_frame
- added link zed_right_camera_optical_frame
Joints:
- added joint zed_camera_center_joint: type fixed, parent base_link, child zed_camera_center, origin xyz=0 0 0 rpy=0 0 0
- added joint zed_left_camera_joint: type fixed, parent zed_camera_center, child zed_left_camera_frame, origin xyz=0 0.06 0 rpy=0 0 0
- added joint zed_left_camera_optical_joint: type fixed, parent zed_left_camera_frame, child zed_left_camera_optical_frame, origin xyz=0 0 0 rpy=-1.57079632679 0.0 -1.57079632679
- added joint zed_right_camera_joint: type fixed, parent zed_camera_center, child zed_right_camera_frame, origin xyz=0 -0.06 0 rpy=0 0 0
- added joint zed_right_camera_optical_joint: type fixed, parent zed_right_camera_frame, child zed_right_camera_optical_frame, origin xyz=0 0 0 rpy=-1.57079632679 0.0 -1.57079632679

Commit message: Drive test and SAR footage changes (#163)
* Add simple publisher and subcriber

* Add ar_track_alvar ros dependency

* Don't fail if can't install catkin_lint

* Add AR tag launch file

* Fix mapper for arm test

* Add ar_track_alvar as dependency in spear_rover

* Ignore vagrant and pycharm files

* Ignore log files

* Move ar launch file

* Rename rover_indiv

* Fix point cloud topic in drive rviz

* Add ar marker visualization to drive rviz

* Fix ar tracker parameters to work in simulation

* Run docker container as privileged

* Add AR markers to test world

* Launch ar track by default in top-level launch files

* Format ar_track.launch

* Remove listener and talker nodes

* Use size of URC markers out of simulator

* Use test world by default

* Fix catkin_lint error

* Add classes to keep track of posts and gates

* Add has_seen to gate

* Fix some marker tracker issues

* Fix python linting

* Remove inaccurate comment

* Add states for testing flexbe properties

* Demo moving to posts and gates

* Add a default tmuxrc

* Use correct ids

* Commit changes and sort it out later

* Get joystick teleop working

* changes

* Fix ros master ip

* Update joystick launch

* Change joystick scales

* Add script to generate ar marker pictures

* Fix dockerfile

* Fix real-world AR tag detection

* Add option to calibrate zed

* Changes

* Add diagnostics publisher node

* Only launch rviz in simulator

* Fix various things

* Misc changes

* Fix spacing

* xml formatting

* Python formatting

Co-authored-by: vyomea <43073294+vyomea@users.noreply.github.com>
Co-authored-by: SPEAR Common <41485825+spearua@users.noreply.github.com>

File: spear_simulator/models/rover/TARS_V2.urdf (robot description, URDF)
Before this commit: robot TARS_V2, 14 links, 13 joints
Links:
- added link zed_camera_center; visual mesh filename=package://zed_wrapper/urdf/models/ZED.stl
- added link zed_left_camera_frame
- added link zed_left_camera_optical_frame
- added link zed_right_camera_frame
- added link zed_right_camera_optical_frame
- link base_link: mass 30.0 -> None
Joints:
- added joint zed_camera_center_joint: type fixed, parent base_link, child zed_camera_center, origin xyz=0 0 0 rpy=0 0 0
- added joint zed_left_camera_joint: type fixed, parent zed_camera_center, child zed_left_camera_frame, origin xyz=0 0.06 0 rpy=0 0 0
- added joint zed_left_camera_optical_joint: type fixed, parent zed_left_camera_frame, child zed_left_camera_optical_frame, origin xyz=0 0 0 rpy=-1.57079632679 0.0 -1.57079632679
- added joint zed_right_camera_joint: type fixed, parent zed_camera_center, child zed_right_camera_frame, origin xyz=0 -0.06 0 rpy=0 0 0
- added joint zed_right_camera_optical_joint: type fixed, parent zed_right_camera_frame, child zed_right_camera_optical_frame, origin xyz=0 0 0 rpy=-1.57079632679 0.0 -1.57079632679

Commit message: Fixed the simulator rover model so that it shows in the simulator

File: spear_simulator/models/rover/TARS_V2.urdf (robot description, URDF)
Before this commit: robot TARS_V2, 19 links, 18 joints
Links:
- link zed_camera_center: geometry 

Commit message: Move wheels to their own urdf

File: spear_simulator/models/rover/TARS_V2.urdf (robot description, URDF)
Before this commit: robot TARS_V2, 19 links, 18 joints
Links:
- removed link link_wheel_backleft
- removed link link_wheel_backright
- removed link link_wheel_frontleft
- removed link link_wheel_frontright
- link zed_camera_center: geometry 
Joints:
- removed joint link_wheel_backleft
- removed joint link_wheel_backright
- removed joint link_wheel_frontleft
- removed joint link_wheel_frontright
