Commit message: Remove unused wheel params

File: spear_simulator/models/rover/wheel.urdf.xacro (robot description, xacro)
@@ -45,11 +45,4 @@
       </joint>
     </transmission>
-    <gazebo reference="link_wheel_${name}">
-      <mu1 value="200.0"/>
-      <mu2 value="100.0"/>
-      <kp value="10000000.0" />
-      <kd value="1.0" />
-      <material>Gazebo/Grey</material>
-    </gazebo>
   </xacro:macro>
 </robot>
