Commit message: Integrate arm into rover model

File: spear_simulator/models/rover/arm.urdf.xacro (robot description, xacro)
@@ -1,12 +1,17 @@
 <?xml version="1.0"?>
 <robot name="arm" xmlns:xacro="http://ros.org/wiki/xacro">
-  <link name="base_link">
-  </link>
   <xacro:property name="shoulder_height" value="0.09" />
   <xacro:property name="bicep_length" value="0.355" />
   <xacro:property name="forearm_length" value="0.185" />
   <xacro:property name="hand_length" value="0.59" />
+  <joint name="arm_mount" type="fixed">
+    <parent link="base_link"/>
+    <child link="arm_mount"/>
+    <origin xyz="0.25 0 0.3"/>
+  </joint>
+  <link name="arm_mount">
+  </link>
   <joint name="shoulder_yaw" type="revolute">
-    <parent link="base_link"/>
+    <parent link="arm_mount"/>
     <child link="shoulder"/>
     <axis xyz="0 0 1"/>

Commit message: Visualize the arm in rviz

File: spear_simulator/models/rover/arm.urdf.xacro (robot description, xacro)
@@ -4,5 +4,20 @@
   <xacro:property name="bicep_length" value="0.355" />
   <xacro:property name="forearm_length" value="0.185" />
+  <xacro:property name="wrist_length" value="${forearm_length/5}" />
+  <xacro:property name="palm_length" value="${forearm_length/4}" />
+  <xacro:property name="finger_length" value="${forearm_length/3}" />
   <xacro:property name="hand_length" value="0.59" />
+  <xacro:property name="arm_width" value="0.05" />
+  <xacro:property name="joint_sep" value="0.005" />
+  <xacro:macro name="arm_link" params="name length">
+    <link name="${name}">
+      <visual>
+        <origin xyz="0 0 ${length/2}" rpy="0 0 0"/>
+        <geometry>
+          <cylinder length="${length-joint_sep}" radius="${arm_width}"/>
+        </geometry>
+      </visual>
+    </link>
+  </xacro:macro>
   <joint name="arm_mount" type="fixed">
     <parent link="base_link"/>
@@ -19,8 +34,5 @@
     <limit lower="-1.58" upper="1.58" effort="1" velocity="0.5"/>
   </joint>
-  <link name="shoulder">
-  </link>
-  <link name="bicep">
-  </link>
+  <arm_link name="shoulder" length="${shoulder_height}"/>
   <joint name="shoulder_pitch" type="revolute">
     <parent link="shoulder"/>
@@ -30,6 +42,5 @@
     <limit lower="0.78" upper="2.15" effort="1" velocity="0.5"/>
   </joint>
-  <link name="forearm">
-  </link>
+  <arm_link name="bicep" length="${bicep_length}"/>
   <joint name="elbow_pitch" type="revolute">
     <parent link="bicep"/>
@@ -39,30 +50,28 @@
     <limit lower="-2.7" upper="1.54" effort="1" velocity="0.5"/>
   </joint>
-  <link name="wrist">
-  </link>
+  <arm_link name="forearm" length="${forearm_length}"/>
   <joint name="wrist_pitch" type="revolute">
     <parent link="forearm"/>
     <child link="wrist"/>
     <axis xyz="0 1 0"/>
-    <origin xyz="0 0 ${forearm_length/5}" rpy="0 0 0"/>
+    <origin xyz="0 0 ${forearm_length}" rpy="0 0 0"/>
     <limit lower="-2.09" upper="2.09" effort="1" velocity="0.5"/>
   </joint>
-  <link name="palm">
-  </link>
+  <arm_link name="wrist" length="${wrist_length}"/>
   <joint name="wrist_roll" type="revolute">
     <parent link="wrist"/>
     <child link="palm"/>
     <axis xyz="0 0 1"/>
-    <origin xyz="0 0 ${forearm_length/4}" rpy="0 0 0"/>
+    <origin xyz="0 0 ${wrist_length}" rpy="0 0 0"/>
     <limit lower="-3" upper="3" effort="1" velocity="0.5"/>
   </joint>
-  <link name="finger">
-  </link>
+  <arm_link name="palm" length="${palm_length}"/>
   <joint name="grab" type="revolute">
     <parent link="palm"/>
     <child link="finger"/>
     <axis xyz="1 0 0"/>
-    <origin xyz="0 0 ${hand_length/3}"/>
+    <origin xyz="0 0 ${palm_length}"/>
     <limit lower="-1" upper="1" effort="1" velocity="0.5"/>
   </joint>
+  <arm_link name="finger" length="${finger_length}"/>
 </robot>

Commit message: Change shoulder range and starting position

File: spear_simulator/models/rover/arm.urdf.xacro (robot description, xacro)
@@ -31,6 +31,6 @@
     <child link="shoulder"/>
     <axis xyz="0 0 1"/>
-    <origin xyz="0 0 0" rpy= "0 0 0"/>
-    <limit lower="-1.58" upper="1.58" effort="1" velocity="0.5"/>
+    <origin xyz="0 0 0" rpy= "0 0 3.14"/>
+    <limit lower="-3.15" upper="3.15" effort="1" velocity="0.5"/>
   </joint>
   <arm_link name="shoulder" length="${shoulder_height}"/>

Commit message: Add an arm controller

File: spear_simulator/models/rover/arm.urdf.xacro (robot description, xacro)
@@ -18,5 +18,25 @@
         </geometry>
       </visual>
+      <inertial>
+        <origin xyz="0 0 ${length/2}" rpy="0 0 0"/>
+        <mass value="0.001" />
+        <inertia ixx="0.001" ixy="0.0" ixz="0.0" iyy="0.001" iyz="0.0" izz="0.001" />
+      </inertial>
     </link>
+  </xacro:macro>
+  <xacro:macro name="arm_joint" params="name **container">
+    <joint name="${name}" type="revolute">
+      <xacro:insert_block name="container"/>
+    </joint>
+    <transmission name="${name}_trans">
+      <type>transmission_interface/SimpleTransmission</type>
+      <actuator name="${name}_actuator">
+        <hardwareInterface>hardware_interface/PositionJointInterface</hardwareInterface>
+        <mechanicalReduction>1</mechanicalReduction>
+      </actuator>
+      <joint name="${name}">
+        <hardwareInterface>hardware_interface/PositionJointInterface</hardwareInterface>
+      </joint>
+    </transmission>
   </xacro:macro>
   <joint name="arm_mount" type="fixed">
@@ -26,6 +46,11 @@
   </joint>
   <link name="arm_mount">
+    <inertial>
+      <origin xyz="0 0 0" rpy="0 0 0" />
+      <mass value="0.001" />
+      <inertia ixx="0.001" ixy="0.0" ixz="0.0" iyy="0.001" iyz="0.0" izz="0.001" />
+    </inertial>
   </link>
-  <joint name="shoulder_yaw" type="revolute">
+  <xacro:arm_joint name="shoulder_yaw"><container>
     <parent link="arm_mount"/>
     <child link="shoulder"/>
@@ -33,7 +58,7 @@
     <origin xyz="0 0 0" rpy= "0 0 3.14"/>
     <limit lower="-3.15" upper="3.15" effort="1" velocity="0.5"/>
-  </joint>
+  </container></xacro:arm_joint>
   <arm_link name="shoulder" length="${shoulder_height}"/>
-  <joint name="shoulder_pitch" type="revolute">
+  <xacro:arm_joint name="shoulder_pitch"><container>
     <parent link="shoulder"/>
     <child link="bicep"/>
@@ -41,7 +66,7 @@
     <origin xyz="0 0 ${shoulder_height}" rpy= "0 0 0"/>
     <limit lower="0.78" upper="2.15" effort="1" velocity="0.5"/>
-  </joint>
+  </container></xacro:arm_joint>
   <arm_link name="bicep" length="${bicep_length}"/>
-  <joint name="elbow_pitch" type="revolute">
+  <xacro:arm_joint name="elbow_pitch"><container>
     <parent link="bicep"/>
     <child link="forearm"/>
@@ -49,7 +74,7 @@
     <origin xyz="0 0 ${bicep_length}" rpy= "0 0 0"/>
     <limit lower="-2.7" upper="1.54" effort="1" velocity="0.5"/>
-  </joint>
+  </container></xacro:arm_joint>
   <arm_link name="forearm" length="${forearm_length}"/>
-  <joint name="wrist_pitch" type="revolute">
+  <xacro:arm_joint name="wrist_pitch"><container>
     <parent link="forearm"/>
     <child link="wrist"/>
@@ -57,7 +82,7 @@
     <origin xyz="0 0 ${forearm_length}" rpy="0 0 0"/>
     <limit lower="-2.09" upper="2.09" effort="1" velocity="0.5"/>
-  </joint>
+  </container></xacro:arm_joint>
   <arm_link name="wrist" length="${wrist_length}"/>
-  <joint name="wrist_roll" type="revolute">
+  <xacro:arm_joint name="wrist_roll"><container>
     <parent link="wrist"/>
     <child link="palm"/>
@@ -65,7 +90,7 @@
     <origin xyz="0 0 ${wrist_length}" rpy="0 0 0"/>
     <limit lower="-3" upper="3" effort="1" velocity="0.5"/>
-  </joint>
+  </container></xacro:arm_joint>
   <arm_link name="palm" length="${palm_length}"/>
-  <joint name="grab" type="revolute">
+  <xacro:arm_joint name="grab"><container>
     <parent link="palm"/>
     <child link="finger"/>
@@ -73,5 +98,5 @@
     <origin xyz="0 0 ${palm_length}"/>
     <limit lower="-1" upper="1" effort="1" velocity="0.5"/>
-  </joint>
+  </container></xacro:arm_joint>
   <arm_link name="finger" length="${finger_length}"/>
 </robot>

Commit message: Add demo IK node

File: spear_simulator/models/rover/arm.urdf.xacro (robot description, xacro)
@@ -43,5 +43,5 @@
     <parent link="base_link"/>
     <child link="arm_mount"/>
-    <origin xyz="0.25 0 0.3"/>
+    <origin xyz="0.25 0 0.3" rpy="0 0 3.1415926535897"/>
   </joint>
   <link name="arm_mount">
@@ -96,5 +96,5 @@
     <child link="finger"/>
     <axis xyz="1 0 0"/>
-    <origin xyz="0 0 ${palm_length}"/>
+    <origin xyz="0 0 ${palm_length}" rpy="0 0 0"/>
     <limit lower="-1" upper="1" effort="1" velocity="0.5"/>
   </container></xacro:arm_joint>

Commit message: Fix arm width vs radius mixup

File: spear_simulator/models/rover/arm.urdf.xacro (robot description, xacro)
@@ -8,5 +8,5 @@
   <xacro:property name="finger_length" value="${forearm_length/3}" />
   <xacro:property name="hand_length" value="0.59" />
-  <xacro:property name="arm_width" value="0.05" />
+  <xacro:property name="arm_width" value="0.1" />
   <xacro:property name="joint_sep" value="0.005" />
   <xacro:macro name="arm_link" params="name length">
@@ -15,5 +15,5 @@
         <origin xyz="0 0 ${length/2}" rpy="0 0 0"/>
         <geometry>
-          <cylinder length="${length-joint_sep}" radius="${arm_width}"/>
+          <cylinder length="${length-joint_sep}" radius="${width/2}"/>
         </geometry>
       </visual>

Commit message: Add fingers to arm

File: spear_simulator/models/rover/arm.urdf.xacro (robot description, xacro)
@@ -10,5 +10,5 @@
   <xacro:property name="arm_width" value="0.1" />
   <xacro:property name="joint_sep" value="0.005" />
-  <xacro:macro name="arm_link" params="name length">
+  <xacro:macro name="arm_link" params="name length width:=${arm_width}">
     <link name="${name}">
       <visual>
@@ -94,9 +94,41 @@
   <xacro:arm_joint name="grab"><container>
     <parent link="palm"/>
-    <child link="finger"/>
+    <child link="grab_placeholder"/>
     <axis xyz="1 0 0"/>
-    <origin xyz="0 0 ${palm_length}" rpy="0 0 0"/>
+    <origin xyz="0 0 0" rpy="0 0 0"/>
     <limit lower="-1" upper="1" effort="1" velocity="0.5"/>
   </container></xacro:arm_joint>
-  <arm_link name="finger" length="${finger_length}"/>
+  <link name="grab_placeholder">
+    <inertial>
+      <mass value="0.001" />
+      <inertia ixx="0.001" ixy="0.0" ixz="0.0" iyy="0.001" iyz="0.0" izz="0.001" />
+    </inertial>
+  </link>
+  <!-- These joints cannot have a transmission, since they are not controlled by gazebo_ros_control -->
+  <joint name="knuckle1" type="revolute">
+    <parent link="palm"/>
+    <child link="finger1"/>
+    <axis xyz="1 0 0"/>
+    <origin xyz="0 0.03 ${palm_length}" rpy="0 0 0"/>
+    <limit lower="-1" upper="1" effort="1" velocity="0.5"/>
+  </joint>
+  <joint name="knuckle2" type="revolute">
+    <parent link="palm"/>
+    <child link="finger2"/>
+    <axis xyz="-1 0 0"/>
+    <origin xyz="0 -0.03 ${palm_length}" rpy="0 0 0"/>
+    <limit lower="-1" upper="1" effort="1" velocity="0.5"/>
+  </joint>
+  <xacro:arm_link name="finger1" length="${finger_length}" width="0.05"/>
+  <xacro:arm_link name="finger2" length="${finger_length}" width="0.05"/>
+  <gazebo>
+    <plugin filename="libroboticsgroup_upatras_gazebo_mimic_joint_plugin.so" name="mimic_joint">
+      <joint>grab</joint>
+      <mimicJoint>knuckle1</mimicJoint>
+    </plugin>
+    <plugin filename="libroboticsgroup_upatras_gazebo_mimic_joint_plugin.so" name="mimic_joint">
+      <joint>grab</joint>
+      <mimicJoint>knuckle2</mimicJoint>
+    </plugin>
+  </gazebo>
 </robot>

Commit message: Add gripper to arm (#240)
* Fix arm width vs radius mixup

* Add fingers to arm

* Skip upatras_gazebo_plugins in catkin_lint

File: spear_simulator/models/rover/arm.urdf.xacro (robot description, xacro)
@@ -8,12 +8,12 @@
   <xacro:property name="finger_length" value="${forearm_length/3}" />
   <xacro:property name="hand_length" value="0.59" />
-  <xacro:property name="arm_width" value="0.05" />
+  <xacro:property name="arm_width" value="0.1" />
   <xacro:property name="joint_sep" value="0.005" />
-  <xacro:macro name="arm_link" params="name length">
+  <xacro:macro name="arm_link" params="name length width:=${arm_width}">
     <link name="${name}">
       <visual>
         <origin xyz="0 0 ${length/2}" rpy="0 0 0"/>
         <geometry>
-          <cylinder length="${length-joint_sep}" radius="${arm_width}"/>
+          <cylinder length="${length-joint_sep}" radius="${width/2}"/>
         </geometry>
       </visual>
@@ -94,9 +94,41 @@
   <xacro:arm_joint name="grab"><container>
     <parent link="palm"/>
-    <child link="finger"/>
+    <child link="grab_placeholder"/>
     <axis xyz="1 0 0"/>
-    <origin xyz="0 0 ${palm_length}" rpy="0 0 0"/>
+    <origin xyz="0 0 0" rpy="0 0 0"/>
     <limit lower="-1" upper="1" effort="1" velocity="0.5"/>
   </container></xacro:arm_joint>
-  <arm_link name="finger" length="${finger_length}"/>
+  <link name="grab_placeholder">
+    <inertial>
+      <mass value="0.001" />
+      <inertia ixx="0.001" ixy="0.0" ixz="0.0" iyy="0.001" iyz="0.0" izz="0.001" />
+    </inertial>
+  </link>
+  <!-- These joints cannot have a transmission, since they are not controlled by gazebo_ros_control -->
+  <joint name="knuckle1" type="revolute">
+    <parent link="palm"/>
+    <child link="finger1"/>
+    <axis xyz="1 0 0"/>
+    <origin xyz="0 0.03 ${palm_length}" rpy="0 0 0"/>
+    <limit lower="-1" upper="1" effort="1" velocity="0.5"/>
+  </joint>
+  <joint name="knuckle2" type="revolute">
+    <parent link="palm"/>
+    <child link="finger2"/>
+    <axis xyz="-1 0 0"/>
+    <origin xyz="0 -0.03 ${palm_length}" rpy="0 0 0"/>
+    <limit lower="-1" upper="1" effort="1" velocity="0.5"/>
+  </joint>
+  <xacro:arm_link name="finger1" length="${finger_length}" width="0.05"/>
+  <xacro:arm_link name="finger2" length="${finger_length}" width="0.05"/>
+  <gazebo>
+    <plugin filename="libroboticsgroup_upatras_gazebo_mimic_joint_plugin.so" name="mimic_joint">
+      <joint>grab</joint>
+      <mimicJoint>knuckle1</mimicJoint>
+    </plugin>
+    <plugin filename="libroboticsgroup_upatras_gazebo_mimic_joint_plugin.so" name="mimic_joint">
+      <joint>grab</joint>
+      <mimicJoint>knuckle2</mimicJoint>
+    </plugin>
+  </gazebo>
 </robot>

Commit message: Initial steps to upgrade to noetic

File: spear_simulator/models/rover/arm.urdf.xacro (robot description, xacro)
@@ -59,5 +59,5 @@
     <limit lower="-3.15" upper="3.15" effort="1" velocity="0.5"/>
   </container></xacro:arm_joint>
-  <arm_link name="shoulder" length="${shoulder_height}"/>
+  <xacro:arm_link name="shoulder" length="${shoulder_height}"/>
   <xacro:arm_joint name="shoulder_pitch"><container>
     <parent link="shoulder"/>
@@ -67,5 +67,5 @@
     <limit lower="0.78" upper="2.15" effort="1" velocity="0.5"/>
   </container></xacro:arm_joint>
-  <arm_link name="bicep" length="${bicep_length}"/>
+  <xacro:arm_link name="bicep" length="${bicep_length}"/>
   <xacro:arm_joint name="elbow_pitch"><container>
     <parent link="bicep"/>
@@ -75,5 +75,5 @@
     <limit lower="-2.7" upper="1.54" effort="1" velocity="0.5"/>
   </container></xacro:arm_joint>
-  <arm_link name="forearm" length="${forearm_length}"/>
+  <xacro:arm_link name="forearm" length="${forearm_length}"/>
   <xacro:arm_joint name="wrist_pitch"><container>
     <parent link="forearm"/>
@@ -83,5 +83,5 @@
     <limit lower="-2.09" upper="2.09" effort="1" velocity="0.5"/>
   </container></xacro:arm_joint>
-  <arm_link name="wrist" length="${wrist_length}"/>
+  <xacro:arm_link name="wrist" length="${wrist_length}"/>
   <xacro:arm_joint name="wrist_roll"><container>
     <parent link="wrist"/>
@@ -91,5 +91,5 @@
     <limit lower="-3" upper="3" effort="1" velocity="0.5"/>
   </container></xacro:arm_joint>
-  <arm_link name="palm" length="${palm_length}"/>
+  <xacro:arm_link name="palm" length="${palm_length}"/>
   <xacro:arm_joint name="grab"><container>
     <parent link="palm"/>

File: spear_simulator/models/rover/wheel.urdf.xacro (robot description, xacro)
@@ -30,5 +30,5 @@
     </link>
     <!-- Stuff to make the wheels driveable -->
-    <joint name="link_wheel_${name}" type="continuous">
+    <joint name="joint_wheel_${name}" type="continuous">
       <axis xyz="0 1 0" rpy="0 0 0"/>
       <origin xyz="${offset}" rpy="0 0 0"/>
@@ -42,5 +42,5 @@
         <mechanicalReduction>1</mechanicalReduction>
       </actuator>
-      <joint name="link_wheel_${name}">
+      <joint name="joint_wheel_${name}">
         <hardwareInterface>hardware_interface/VelocityJointInterface</hardwareInterface>
       </joint>
