Commit message: Split cameras into separate files and add webcams

File: pkg/spear_simulator/models/rover/TARS_V2.urdf.xacro (robot description, xacro)
@@ -2,56 +2,10 @@
 <!-- created with Phobos 0.8 -->
   <robot name="TARS_V2" xmlns:xacro="http://ros.org/wiki/xacro">
+    <xacro:include filename="$(find spear_simulator)/models/rover/constants.xacro"/>
     <xacro:include filename="$(find spear_simulator)/models/rover/wheel.urdf.xacro"/>
     <xacro:include filename="$(find spear_simulator)/models/rover/arm.urdf.xacro"/>
-    <xacro:property name="M_PI" value="3.1415926535897" />
-    <xacro:property name="WHEEL_SEP_LENGTH" value="0.44"/>
-    <xacro:property name="WHEEL_SEP_WIDTH" value="0.44"/>
-    <link name="link_camera_back">
-    </link>
-    <link name="link_camera_depth">
-    </link>
-    <link name="camera_depth_optical_frame">
-    </link>
+    <xacro:include filename="$(find spear_simulator)/models/rover/zed_cam.urdf.xacro"/>
+    <xacro:include filename="$(find spear_simulator)/models/rover/webcam.urdf.xacro"/>
     <link name="imu_link">
-    </link>
-    <gazebo reference="link_camera_depth">
-      <sensor type="depth" name="camera_depth">
-        <always_on>true</always_on>
-        <update_rate>20.0</update_rate>
-        <camera>
-          <!-- Set camera geometry based on zed cam at 720p -->
-          <!-- 70 degress fov -->
-          <horizontal_fov>1.2217</horizontal_fov>
-          <image>
-            <format>B8G8R8</format>
-            <width>1280</width>
-            <height>720</height>
-          </image>
-          <clip>
-            <near>0.05</near>
-            <far>8.0</far>
-          </clip>
-        </camera>
-        <plugin name="kinect_camera_controller" filename="libgazebo_ros_openni_kinect.so">
-          <cameraName>camera_depth</cameraName>
-          <alwaysOn>true</alwaysOn>
-          <updateRate>100</updateRate>
-          <imageTopicName>rgb/image_raw</imageTopicName>
-          <depthImageTopicName>depth/image_raw</depthImageTopicName>
-          <pointCloudTopicName>depth/points</pointCloudTopicName>
-          <cameraInfoTopicName>rgb/camera_info</cameraInfoTopicName>
-          <depthImageCameraInfoTopicName>depth/camera_info</depthImageCameraInfoTopicName>
-          <frameName>camera_depth_optical_frame</frameName>
-          <baseline>0.1</baseline>
-          <distortion_k1>0.0</distortion_k1>
-          <distortion_k2>0.0</distortion_k2>
-          <distortion_k3>0.0</distortion_k3>
-          <distortion_t1>0.0</distortion_t1>
-          <distortion_t2>0.0</distortion_t2>
-          <pointCloudCutoff>0.4</pointCloudCutoff>
-        </plugin>
-      </sensor>
-    </gazebo>
-    <link name="link_camera_front">
     </link>
     <link name="base_link">
@@ -154,28 +108,13 @@
     <xacro:wheel side="left" name="backleft" offset="${-WHEEL_SEP_LENGTH/2} ${WHEEL_SEP_WIDTH/2} 0"/>
     <xacro:wheel side="right" name="backright" offset="${-WHEEL_SEP_LENGTH/2} ${-WHEEL_SEP_WIDTH/2} 0"/>
-    <joint name="link_camera_back" type="fixed">
-      <origin xyz="-0.315 1e-05 0.3439" rpy="3.14159 1.5708 0"/>
-      <parent link="base_link"/>
-      <child link="link_camera_back"/>
-    </joint>
-    <joint name="link_camera_depth" type="fixed">
-      <origin xyz="0.3 0 0.2" rpy="0 0 0"/>
-      <parent link="base_link"/>
-      <child link="link_camera_depth"/>
-    </joint>
-    <joint name="camera_depth_optical_frame" type="fixed">
-      <origin xyz="0 0 0" rpy="${-M_PI/2} 0 ${-M_PI/2}"/>
-      <parent link="link_camera_depth"/>
-      <child link="camera_depth_optical_frame"/>
-    </joint>
+    <xacro:zed_cam xyz="0.3 0 0.2" rpy="0 0 0"/>
+    <xacro:webcam name="front" xyz="0.315 -0.11999 0.3439" rpy="0 0 0"/>
+    <xacro:webcam name="back" xyz="-0.315 1e-05 0.3439" rpy="0 0 ${M_PI}"/>
+    <xacro:webcam name="left" xyz="0 0.24 0.3439" rpy="0 0 ${M_PI/2}"/>
+    <xacro:webcam name="right" xyz="0 -0.24 0.3439" rpy="0 0 ${-M_PI/2}"/>
     <joint name="imu_link" type="fixed">
       <origin xyz="0 0 0.2" rpy="0 0 0"/>
       <parent link="base_link"/>
       <child link="imu_link"/>
-    </joint>
-    <joint name="link_camera_front" type="fixed">
-      <origin xyz="0.315 -0.11999 0.3439" rpy="0 1.5708 0"/>
-      <parent link="base_link"/>
-      <child link="link_camera_front"/>
     </joint>
     <joint name="link_suspension_backleft" type="fixed">
@@ -236,37 +175,3 @@
       </sensor>
     </gazebo>
-    <!-- Camera Center -->
-    <joint name="zed_camera_center_joint" type="fixed">
-        <parent link="base_link"/>
-        <child link="zed_camera_center"/>
-        <origin xyz="0 0 0" rpy="0 0 0" />
-    </joint>
-    <link name="zed_camera_center">
-    </link>
-<!-- Left Camera -->
-    <joint name="zed_left_camera_joint" type="fixed">
-        <parent link="zed_camera_center"/>
-        <child link="zed_left_camera_frame"/>
-        <origin xyz="0 0.06 0" rpy="0 0 0" />
-    </joint>
-    <link name="zed_left_camera_frame" />
-    <joint name="zed_left_camera_optical_joint" type="fixed">
-        <origin xyz="0 0 0" rpy="-1.57079632679 0.0 -1.57079632679"/>
-        <parent link="zed_left_camera_frame"/>
-        <child link="zed_left_camera_optical_frame"/>
-    </joint>
-    <link name="zed_left_camera_optical_frame"/>
-<!-- Right Camera -->
-    <joint name="zed_right_camera_joint" type="fixed">
-        <parent link="zed_camera_center"/>
-        <child link="zed_right_camera_frame"/>
-        <origin xyz="0 -0.06 0" rpy="0 0 0" />
-    </joint>
-    <link name="zed_right_camera_frame" />
-    <joint name="zed_right_camera_optical_joint" type="fixed">
-        <origin xyz="0 0 0" rpy="-1.57079632679 0.0 -1.57079632679"/>
-        <parent link="zed_right_camera_frame"/>
-        <child link="zed_right_camera_optical_frame"/>
-    </joint>
-    <link name="zed_right_camera_optical_frame"/>
   </robot>

File: pkg/spear_simulator/models/rover/wheel.urdf.xacro (robot description, xacro)
@@ -1,4 +1,5 @@
 <?xml version="1.0"?>
 <robot name="wheel" xmlns:xacro="http://ros.org/wiki/xacro">
+  <xacro:include filename="$(find spear_simulator)/models/rover/constants.xacro"/>
   <xacro:macro name="wheel" params="name side offset">
     <xacro:property name="link_origin" value="0 0 0"/>
